Commit message: action 오류 수정, 물체 초기값 동적 지정

File: g1_pnp_generator/assets/robots/g1_29dof_with_3finger.urdf (robot description, URDF)
Before this commit: robot g1_29dof_with_hand, 54 links, 53 joints
Joints:
- joint waist_pitch_joint: limit lower=-0.3 upper=0.3 effort=50 velocity=37 -> lower=-0.5 upper=0.5 effort=50 velocity=37
- joint waist_roll_joint: limit lower=-0.3 upper=0.3 effort=50 velocity=37 -> lower=-0.5 upper=0.5 effort=50 velocity=37
- joint waist_yaw_joint: limit lower=-1 upper=1 effort=88 velocity=32 -> lower=-1.5 upper=1.5 effort=88 velocity=32
